Commit message: First URDF version.

File: quetzal.urdf (robot description, URDF)
Before this commit: robot robot_name, 4 links, 3 joints
Links:
- added link link2; visual mesh filename=package://QuetzalArmURDF/meshes/link.dae
- added link link3; visual mesh filename=package://QuetzalArmURDF/meshes/link.dae
- added link link4; visual mesh filename=package://QuetzalArmURDF/meshes/link.dae
- added link link5; visual mesh filename=package://QuetzalArmURDF/meshes/link.dae
- added link link6; visual mesh filename=package://QuetzalArmURDF/meshes/link.dae
- added link link7; visual mesh filename=package://QuetzalArmURDF/meshes/link.dae
- added link link8; visual mesh filename=package://QuetzalArmURDF/meshes/link.dae
- added link link9; visual mesh filename=package://QuetzalArmURDF/meshes/link.dae
Joints:
- added joint joint1: type spherical, parent link1, child link2, origin xyz=0 0 0.1
- added joint joint2: type spherical, parent link2, child link3, origin xyz=0 0 0.1
- added joint joint3: type spherical, parent link3, child link4, origin xyz=0 0 0.1
- added joint joint4: type spherical, parent link4, child link5, origin xyz=0 0 0.1
- added joint joint5: type spherical, parent link5, child link6, origin xyz=0 0 0.1
- added joint joint6: type spherical, parent link6, child link7, origin xyz=0 0 0.1
- added joint joint7: type spherical, parent link7, child link8, origin xyz=0 0 0.1
- added joint joint8: type spherical, parent link8, child link9, origin xyz=0 0 0.1

Commit message: New URDF added.

File: quetzal.urdf (robot description, URDF)
Before this commit: robot robot_name, 12 links, 11 joints
Joints:
- joint end_effector_joint: origin xyz=0 0 0.1 -> xyz=0.1 0.0 0.0
- joint joint0: origin xyz=0 0 0 -> xyz=0 0 0.1 rpy=0 -1.5707 0 
- joint joint1: origin xyz=0 0 0.1 -> xyz=0.1 0.0 0.0
- joint joint2: origin xyz=0 0 0.1 -> xyz=0.1 0.0 0.0
- joint joint3: origin xyz=0 0 0.1 -> xyz=0.1 0.0 0.0
- joint joint4: origin xyz=0 0 0.1 -> xyz=0.1 0.0 0.0
- joint joint5: origin xyz=0 0 0.1 -> xyz=0.1 0.0 0.0
- joint joint6: origin xyz=0 0 0.1 -> xyz=0.1 0.0 0.0
- joint joint7: origin xyz=0 0 0.1 -> xyz=0.1 0.0 0.0
- joint joint8: origin xyz=0 0 0.1 -> xyz=0.1 0.0 0.0
- joint joint9: origin xyz=0 0 0.1 -> xyz=0.1 0.0 0.0
